Commit message: fixed pathing for urdf

File: digbot4/urdf/digbot4.urdf (robot description, URDF)
Before this commit: robot digbot4, 11 links, 10 joints
Links:
- link base_link: geometry collision mesh filename=package://lunabotics/digbot4/meshes/base_link.STL; visual mesh filename=package://lunabotics/digbot4/meshes/base_link.STL
- link front_cam: geometry collision mesh filename=package://lunabotics/digbot4/meshes/front_cam.STL; visual mesh filename=package://lunabotics/digbot4/meshes/front_cam.STL
- link front_cam_mount: geometry collision mesh filename=package://lunabotics/digbot4/meshes/front_cam_mount.STL; visual mesh filename=package://lunabotics/digbot4/meshes/front_cam_mount.STL
- link front_left_wheel: geometry collision mesh filename=package://lunabotics/digbot4/meshes/front_left_wheel.STL; visual mesh filename=package://lunabotics/digbot4/meshes/front_left_wheel.STL
- link front_lidar: geometry collision mesh filename=package://lunabotics/digbot4/meshes/front_lidar.STL; visual mesh filename=package://lunabotics/digbot4/meshes/front_lidar.STL
- link front_right_wheel: geometry collision mesh filename=package://lunabotics/digbot4/meshes/front_right_wheel.STL; visual mesh filename=package://lunabotics/digbot4/meshes/front_right_wheel.STL
- link rear_cam: geometry collision mesh filename=package://lunabotics/digbot4/meshes/rear_cam.STL; visual mesh filename=package://lunabotics/digbot4/meshes/rear_cam.STL
- link rear_cam_mount: geometry collision mesh filename=package://lunabotics/digbot4/meshes/rear_cam_mount.STL; visual mesh filename=package://lunabotics/digbot4/meshes/rear_cam_mount.STL
- link rear_left_wheel: geometry collision mesh filename=package://lunabotics/digbot4/meshes/rear_left_wheel.STL; visual mesh filename=package://lunabotics/digbot4/meshes/rear_left_wheel.STL
- link rear_lidar: geometry collision mesh filename=package://lunabotics/digbot4/meshes/rear_lidar.STL; visual mesh filename=package://lunabotics/digbot4/meshes/rear_lidar.STL
- link rear_right_wheel: geometry collision mesh filename=package://lunabotics/digbot4/meshes/rear_right_wheel.STL; visual mesh filename=package://lunabotics/digbot4/meshes/rear_right_wheel.STL

Commit message: drive plugin working

File: digbot4/urdf/digbot4.urdf (robot description, URDF)
Before this commit: robot digbot4, 11 links, 10 joints
Joints:
- joint front_left_wheel_joint: axis 0 -1 0 -> 0 1 0
- joint front_right_wheel_joint: axis 0 -1 0 -> 0 1 0
